Commit message: Update lidar.xacro

File: speedy_duck/description/lidar.xacro (robot description, xacro)
@@ -4,5 +4,5 @@
         <parent link="chassis"/>
         <child link="laser_frame"/>
-        <origin xyz="0.122 0 0.212" rpy="0 0 0"/>
+        <origin xyz="0.2 0 0.18" rpy="0 0 0"/>
     </joint>
     <link name="laser_frame">
